File: shematics/kicad/RcOid/RcOid/RcOid.kicad_pcb (KiCad board)
At the start: 2 copper layers, 30 x 26 mm, 9 parts, among them J1 Wemos Left (5V), J2 Wemos Right (3.3V), Q1 IRLU024N, U1 TSOP531xx

Commit message: fix PCB wrong Footprint
Parts:
- Q1: footprint Package_TO_SOT_THT:TO-251-2-1EP_Horizontal_TabDown -> Package_TO_SOT_THT:TO-251-3-1EP_Horizontal_TabDown
Routing:
- net GND: track 74.8 -> 69.0 mm
- net Net-(D1-Pad1): track 13.1 -> 12.2 mm
