File: shematics/kicad/RcOid/RcOid/RcOid.sch (KiCad schematic (older format))
At the start: 7 parts, among them J1 Wemos Left (5V), J2 Wemos Right (3.3V), U1 TSOP531xx

Commit message: Schematc Update
Parts:
- gave numbers to parts that had none: 1
Changed lines of the file:
@@
 Sheet 1 1
 Title "RcOid Ir Schaltung"
-Date "2020-10-30"
-Rev "1"
-Comp ""
+Date "2020-11-08"
+Rev "2"
+Comp "smart-devices.cf"
 Comment1 ""
 Comment2 ""
@@
 	3100 4350 2450 4350
 $Comp
-L Device:Q_NMOS_GDS Q?
+L Device:Q_NMOS_GDS Q1
 U 1 1 5FA71831
 P 3850 3100
-F 0 "Q?" H 4054 3146 50  0000 L CNN
+F 0 "Q1" H 4054 3146 50  0000 L CNN
 F 1 "IRLU024N" H 4054 3055 50  0000 L CNN
 F 2 "" H 4050 3200 50  0001 C CNN

Commit message: change R
Parts:
- R1: value 47 -> 10
Changed lines of the file:
@@
 P 3950 1900
 F 0 "R1" H 4020 1946 50  0000 L CNN
-F 1 "47" H 4020 1855 50  0000 L CNN
+F 1 "10" H 4020 1855 50  0000 L CNN
 F 2 "Resistor_THT:R_Axial_DIN0411_L9.9mm_D3.6mm_P15.24mm_Horizontal" V 3880 1900 50  0001 C CNN
 F 3 "~" H 3950 1900 50  0001 C CNN

Commit message: TH PCB
Parts:
- added D2: TRU 1577326, LED_THT:LED_D5.0mm_IRGrey, symbol LED:LD274
- added JP1: SJ, Jumper:SolderJumper-2_P1.3mm_Open_Pad1.0x1.5mm, symbol Jumper:SolderJumper_2_Open
- C1: value 3000µF -> 2000µF
- D1: value LD271 -> TRU 1577326; footprint LED_THT:LED_D5.0mm_IRGrey -> LED_THT:LED_D5.0mm_Horizontal_O1.27mm_Z3.0mm_IRGrey
- Q1: footprint (none) -> Package_TO_SOT_THT:TO-251-2-1EP_Horizontal_TabDown
- R1: value 10 -> 47
Connections:
- net at D1.2 (A): now also D2.1 (K), JP1.2 (B); no longer R1.2
- new net: D2.2 (A), JP1.1 (A), R1.2
Changed lines of the file:
@@
 Sheet 1 1
 Title "RcOid Ir Schaltung"
-Date "2020-11-08"
-Rev "2"
-Comp "smart-devices.cf"
+Date "2020-10-30"
+Rev "1"
+Comp ""
 Comment1 ""
 Comment2 ""
@@
 P 3950 1900
 F 0 "R1" H 4020 1946 50  0000 L CNN
-F 1 "10" H 4020 1855 50  0000 L CNN
+F 1 "47" H 4020 1855 50  0000 L CNN
 F 2 "Resistor_THT:R_Axial_DIN0411_L9.9mm_D3.6mm_P15.24mm_Horizontal" V 3880 1900 50  0001 C CNN
 F 3 "~" H 3950 1900 50  0001 C CNN
@@
 P 3950 2600
 F 0 "D1" V 3946 2520 50  0000 R CNN
-F 1 "LD271" V 3855 2520 50  0000 R CNN
-F 2 "LED_THT:LED_D5.0mm_IRGrey" H 3950 2775 50  0001 C CNN
+F 1 "TRU 1577326" V 3855 2520 50  0000 R CNN
+F 2 "LED_THT:LED_D5.0mm_Horizontal_O1.27mm_Z3.0mm_IRGrey" H 3950 2775 50  0001 C CNN
 F 3 "http://www.alliedelec.com/m/d/40788c34903a719969df15f1fbea1056.pdf" H 3900 2600 50  0001 C CNN
 	1    3950 2600
 	0    -1   -1   0
 $EndComp
-Wire Wire Line
-	3950 2050 3950 2500
 Wire Wire Line
 	3950 2800 3950 2900
@@
 P 4650 3700
 F 0 "C1" H 4532 3654 50  0000 R CNN
-F 1 "3000µF" H 4532 3745 50  0000 R CNN
+F 1 "2000µF" H 4532 3745 50  0000 R CNN
 F 2 "Capacitor_THT:CP_Radial_D10.0mm_P2.50mm" H 4688 3550 50  0001 C CNN
 F 3 "~" H 4650 3700 50  0001 C CNN
@@
 F 0 "Q1" H 4054 3146 50  0000 L CNN
 F 1 "IRLU024N" H 4054 3055 50  0000 L CNN
-F 2 "" H 4050 3200 50  0001 C CNN
+F 2 "Package_TO_SOT_THT:TO-251-2-1EP_Horizontal_TabDown" H 4050 3200 50  0001 C CNN
 F 3 "~" H 3850 3100 50  0001 C CNN
 	1    3850 3100
 	1    0    0    -1
 $EndComp
+$Comp
+L LED:LD274 D2
+U 1 1 5FAC439D
+P 3950 2200
+F 0 "D2" V 3946 2121 50  0000 R CNN
+F 1 "TRU 1577326" V 3855 2121 50  0000 R CNN
+F 2 "LED_THT:LED_D5.0mm_IRGrey" H 3950 2375 50  0001 C CNN
+F 3 "http://pdf.datasheetcatalog.com/datasheet/siemens/LD274.pdf" H 3900 2200 50  0001 C CNN
+	1    3950 2200
+	0    -1   -1   0
+$EndComp
+Wire Wire Line
+	3950 2050 3950 2100
+Wire Wire Line
+	3950 2400 3950 2500
+$Comp
+L Jumper:SolderJumper_2_Open JP1
+U 1 1 5FAC6616
+P 3550 2250
+F 0 "JP1" V 3504 2318 50  0000 L CNN
+F 1 "SJ" V 3595 2318 50  0000 L CNN
+F 2 "Jumper:SolderJumper-2_P1.3mm_Open_Pad1.0x1.5mm" H 3550 2250 50  0001 C CNN
+F 3 "~" H 3550 2250 50  0001 C CNN
+	1    3550 2250
+	0    1    1    0
+$EndComp
+Wire Wire Line
+	3550 2100 3950 2100
+Connection ~ 3950 2100
+Wire Wire Line
+	3550 2400 3950 2400
+Connection ~ 3950 2400
 $EndSCHEMATC

Commit message: Werte aktualisiert
Parts:
- D1, D2: value TRU 1577326 -> TSAL6400
- R1: value 47 -> 2.4
- U1: value TSOP531xx -> VS1838B
Changed lines of the file:
@@
 EESchema Schematic File Version 4
+LIBS:RcOid-cache
 EELAYER 30 0
 EELAYER END
@@
 P 3950 1900
 F 0 "R1" H 4020 1946 50  0000 L CNN
-F 1 "47" H 4020 1855 50  0000 L CNN
+F 1 "2.4" H 4020 1855 50  0000 L CNN
 F 2 "Resistor_THT:R_Axial_DIN0411_L9.9mm_D3.6mm_P15.24mm_Horizontal" V 3880 1900 50  0001 C CNN
 F 3 "~" H 3950 1900 50  0001 C CNN
@@
 P 2600 2650
 F 0 "U1" H 2588 3075 50  0000 C CNN
-F 1 "TSOP531xx" H 2588 2984 50  0000 C CNN
+F 1 "VS1838B" H 2588 2984 50  0000 C CNN
 F 2 "OptoDevice:Vishay_MINIMOLD-3Pin" H 2550 2275 50  0001 C CNN
 F 3 "http://www.vishay.com/docs/82745/tsop531.pdf" H 3250 2950 50  0001 C CNN
@@
 P 3950 2600
 F 0 "D1" V 3946 2520 50  0000 R CNN
-F 1 "TRU 1577326" V 3855 2520 50  0000 R CNN
+F 1 "TSAL6400" V 3855 2520 50  0000 R CNN
 F 2 "LED_THT:LED_D5.0mm_Horizontal_O1.27mm_Z3.0mm_IRGrey" H 3950 2775 50  0001 C CNN
 F 3 "http://www.alliedelec.com/m/d/40788c34903a719969df15f1fbea1056.pdf" H 3900 2600 50  0001 C CNN
@@
 P 3950 2200
 F 0 "D2" V 3946 2121 50  0000 R CNN
-F 1 "TRU 1577326" V 3855 2121 50  0000 R CNN
+F 1 "TSAL6400" V 3855 2121 50  0000 R CNN
 F 2 "LED_THT:LED_D5.0mm_IRGrey" H 3950 2375 50  0001 C CNN
 F 3 "http://pdf.datasheetcatalog.com/datasheet/siemens/LD274.pdf" H 3900 2200 50  0001 C CNN
